File: pcb/skydrop.sch (EAGLE design)
At the start: 99 parts, among them IC1 RT9193-33GB, IC2 MCP73831/OT, IC3 STM809SWX6F, IC4 MS5611-01BA03, Q1 BSS84, Q10 BSS84, Q2 BSS123, Q3 BSS123, Q4 BSS84, Q5 BSS84, Q6 BSS84, Q7 BSS123, Q8 BSS84, Q9 BSS84, U2 W25Q16BVSS

Commit message: start spi flash support
Parts:
- removed C11, C17: (no value), skydrop:C_0805
- removed C15: (no value), skydrop:C_1210
- removed C16, C22: 0.01uf, skydrop:C_0805
- removed D3, D4: (no value), skydrop:DIODE_SOD-123FL
- removed JP2: (no value), skydrop:PINHD-1X8
- removed Q10, Q9: BSS84, transistor-small-signal:BSS84
- removed R10, R28, R33, R37: 10k, skydrop:R_0805
- removed R3, R35, R36, R39: 0, skydrop:R_1206
- removed R38: 100, skydrop:R_0805
- removed R40, R41, R42, R43: 47k, skydrop:R_0805
- removed U2: W25Q16BVSS, skydrop:W25Q16BVSS
- added C6: (no value), skydrop:C_0805
- JP3: device pinhead:PINHD-1X4 -> pinhead:PINHD-1X12
- R2: device skydrop:R_1206 -> skydrop:R_0805
- R23: value 100 -> 0; device skydrop:R_0805 -> skydrop:R_1206
- R31: value 10k -> 0; device skydrop:R_0805 -> skydrop:R_1206
- R8: value 3.3k -> (none)
- R9: value 10k -> (none)
- U1: device skydrop:GPS_FGPMMOPA6C -> adafruit:GPS_FGPMMOPA6H
Connections:
- removed net BTN_C_B1: C22.1, R42.1
- removed net FLASH_CLK: U2.CLK, UC1.PB13/SPI2_SCK/USART3_CTS/TIM1_CH1N
- removed net FLASH_CS: R28.1, U2.!CS!, UC1.PB12/SPI2_NSS/I2C2_SMBAL/USART3_CK/TIM1_BKIN
- removed net FLASH_DI: U2.DI, UC1.PB15/SPI2_MOSI/TIM1_CH3N
- removed net FLASH_DO: U2.DO, UC1.PB14/SPI2_MISO/USART3_RTS/TIM1_CH2N
- removed net GPS_3D_FIX: U1.3D-FIX, UC1.PA1/USART2_RTS/ADC1/TIM2_CH2
- removed net GPS_PWR: R23.2, UC1.PC3/ADC13
- removed net GPS_RX: U1.RX, UC1.PA2/USART2_TX/ADC2/TIM2_CH3
- removed net GPS_TX: R3.2, UC1.PA3/USART2_RX/ADC3/TIM2_CH4
- removed net N$1: Q5.S, Q6.S, R11.2, R12.2, R2.1
- removed net N$17: R3.1, U1.TX
- removed net N$18: Q9.G, R10.1, R23.1
- removed net N$28: R31.1, U2.!WP!
- removed net N$37: C17.2, R28.2, R31.2, R33.2, R35.1, U2.VCC
- removed net N$38: R36.2, R6.2, R7.1
- removed net N$39: Q10.G, R37.1, R38.1
- removed net N$43: Q10.D, R15.1
- removed net N$44: JP3.4, R39.1
- removed net N$45: C16.2, D4.A, R41.1
- removed net N$46: C22.2, D3.A, R43.1
- removed net USB_CON: R38.2, UC1.PC10
- removed net USB_VBUS: R8.2, R9.1, UC1.PA10/USART1_RX/TIM1_CH3
- removed net WAKE_UP: D3.C, D4.C, R34.2, UC1.PA0-WKUP/USART2_CTS/ADC0/TIM2_CH1_ETR
- new net SND_1N: UC1.PB13/SPI2_SCK/USART3_CTS/TIM1_CH1N
- new net SND_2N: UC1.PB14/SPI2_MISO/USART3_RTS/TIM1_CH2N
- new net USB_U: R31.1, R8.2, R9.1, UC1.PA10/USART1_RX/TIM1_CH3
- net +5V: now also R15.1
- net BAT_EN: now also UC1.PB12/SPI2_NSS/I2C2_SMBAL/USART3_CK/TIM1_BKIN; no longer UC1.PC6
- net BAT_SNS: now also R6.2, R7.1; no longer R36.1
- net BTN_C_B: now also C6.2, JP3.12, R34.2, UC1.PA0-WKUP/USART2_CTS/ADC0/TIM2_CH1_ETR; no longer C16.1, JP3.3, R40.1, UC1.PC2/ADC12
- net BTN_L_B: now also JP3.11, UC1.PA1/USART2_RTS/ADC1/TIM2_CH2; no longer JP3.2, UC1.PC1/ADC11
- net BTN_R_B: now also JP3.10, UC1.PA2/USART2_TX/ADC2/TIM2_CH3; no longer JP3.1, UC1.PC0/ADC10
- net CHARGE_STAT: now also R23.2; no longer IC2.STAT
- net GND: now also JP3.2; no longer C11.2, C15.2, C17.1, JP2.1, R40.2, R41.2, R42.2, R43.2, U1.GND@1, U2.GND
- net LCD_CE_B: now also JP3.3; no longer JP2.2
- net LCD_CLK_B: now also JP3.7; no longer JP2.6
- net LCD_DC_B: now also JP3.4; no longer JP2.3
- net LCD_DIN_B: now also JP3.6; no longer JP2.5
- net LCD_PWR_B: now also JP3.5; no longer JP2.4
- net LCD_RST_B: now also JP3.8; no longer JP2.7
- net N$23: now also IC2.STAT, R23.1; no longer R33.1, U2.!HOLD!
- net N$30: now also C6.1, R31.2; no longer Q9.D, U1.VCC
- net N$5: now also R2.2
- net SND_PWR: now also Q5.S, Q6.S, R11.2, R12.2, R2.1; no longer C11.1, C15.1, R2.2
- net VCC: now also JP3.9; no longer JP2.8, Q10.S, Q9.S, R10.2, R35.2, R37.2, R39.2, U1.VBACKUP
Other:
- note added: "USB WakeUP"
- note added: "place if have no power supervisor"
- moved on the sheet: C12, C13, C19, C20, C3, C4, C5, IC1, IC3, J1, JP4, JP6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

Commit message: pcb improovment, gitignore change
Parts:
- removed C6: (no value), skydrop:C_0805
- added C11, C17: (no value), skydrop:C_0805
- added C15: (no value), skydrop:C_1210
- added C16, C22: 0.01uf, skydrop:C_0805
- added D3, D4: (no value), skydrop:DIODE_SOD-123FL
- added JP2: (no value), skydrop:PINHD-1X8
- added Q10, Q9: BSS84, transistor-small-signal:BSS84
- added R10, R28, R33, R37: 10k, skydrop:R_0805
- added R3, R35, R36, R39: 0, skydrop:R_1206
- added R38: 100, skydrop:R_0805
- added R40, R41, R42, R43: 47k, skydrop:R_0805
- added U2: W25Q16BVSS, skydrop:W25Q16BVSS
- JP3: device pinhead:PINHD-1X12 -> pinhead:PINHD-1X4
- R2: device skydrop:R_0805 -> skydrop:R_1206
- R23: value 0 -> 100; device skydrop:R_1206 -> skydrop:R_0805
- R31: value 0 -> 10k; device skydrop:R_1206 -> skydrop:R_0805
- R8: value (none) -> 3.3k
- R9: value (none) -> 10k
- U1: device adafruit:GPS_FGPMMOPA6H -> skydrop:GPS_FGPMMOPA6C
Connections:
- removed net SND_1N: UC1.PB13/SPI2_SCK/USART3_CTS/TIM1_CH1N
- removed net SND_2N: UC1.PB14/SPI2_MISO/USART3_RTS/TIM1_CH2N
- removed net USB_U: R31.1, R8.2, R9.1, UC1.PA10/USART1_RX/TIM1_CH3
- new net BTN_C_B1: C22.1, R42.1
- new net FLASH_CLK: U2.CLK, UC1.PB13/SPI2_SCK/USART3_CTS/TIM1_CH1N
- new net FLASH_CS: R28.1, U2.!CS!, UC1.PB12/SPI2_NSS/I2C2_SMBAL/USART3_CK/TIM1_BKIN
- new net FLASH_DI: U2.DI, UC1.PB15/SPI2_MOSI/TIM1_CH3N
- new net FLASH_DO: U2.DO, UC1.PB14/SPI2_MISO/USART3_RTS/TIM1_CH2N
- new net GPS_3D_FIX: U1.3D-FIX, UC1.PA1/USART2_RTS/ADC1/TIM2_CH2
- new net GPS_PWR: R23.2, UC1.PC3/ADC13
- new net GPS_RX: U1.RX, UC1.PA2/USART2_TX/ADC2/TIM2_CH3
- new net GPS_TX: R3.2, UC1.PA3/USART2_RX/ADC3/TIM2_CH4
- new net N$1: Q5.S, Q6.S, R11.2, R12.2, R2.1
- new net N$17: R3.1, U1.TX
- new net N$18: Q9.G, R10.1, R23.1
- new net N$28: R31.1, U2.!WP!
- new net N$37: C17.2, R28.2, R31.2, R33.2, R35.1, U2.VCC
- new net N$38: R36.2, R6.2, R7.1
- new net N$39: Q10.G, R37.1, R38.1
- new net N$43: Q10.D, R15.1
- new net N$44: JP3.4, R39.1
- new net N$45: C16.2, D4.A, R41.1
- new net N$46: C22.2, D3.A, R43.1
- new net USB_CON: R38.2, UC1.PC10
- new net USB_VBUS: R8.2, R9.1, UC1.PA10/USART1_RX/TIM1_CH3
- new net WAKE_UP: D3.C, D4.C, R34.2, UC1.PA0-WKUP/USART2_CTS/ADC0/TIM2_CH1_ETR
- net +5V: no longer R15.1
- net BAT_EN: now also UC1.PC6; no longer UC1.PB12/SPI2_NSS/I2C2_SMBAL/USART3_CK/TIM1_BKIN
- net BAT_SNS: now also R36.1; no longer R6.2, R7.1
- net BTN_C_B: now also C16.1, JP3.3, R40.1, UC1.PC2/ADC12; no longer C6.2, JP3.12, R34.2, UC1.PA0-WKUP/USART2_CTS/ADC0/TIM2_CH1_ETR
- net BTN_L_B: now also JP3.2, UC1.PC1/ADC11; no longer JP3.11, UC1.PA1/USART2_RTS/ADC1/TIM2_CH2
- net BTN_R_B: now also JP3.1, UC1.PC0/ADC10; no longer JP3.10, UC1.PA2/USART2_TX/ADC2/TIM2_CH3
- net CHARGE_STAT: now also IC2.STAT; no longer R23.2
- net GND: now also C11.2, C15.2, C17.1, JP2.1, R40.2, R41.2, R42.2, R43.2, U1.GND@1, U2.GND; no longer JP3.2
- net LCD_CE_B: now also JP2.2; no longer JP3.3
- net LCD_CLK_B: now also JP2.6; no longer JP3.7
- net LCD_DC_B: now also JP2.3; no longer JP3.4
- net LCD_DIN_B: now also JP2.5; no longer JP3.6
- net LCD_PWR_B: now also JP2.4; no longer JP3.5
- net LCD_RST_B: now also JP2.7; no longer JP3.8
- net N$23: now also R33.1, U2.!HOLD!; no longer IC2.STAT, R23.1
- net N$30: now also Q9.D, U1.VCC; no longer C6.1, R31.2
- net N$5: no longer R2.2
- net SND_PWR: now also C11.1, C15.1, R2.2; no longer Q5.S, Q6.S, R11.2, R12.2, R2.1
- net VCC: now also JP2.8, Q10.S, Q9.S, R10.2, R35.2, R37.2, R39.2, U1.VBACKUP; no longer JP3.9
Other:
- note removed: "USB WakeUP"
- note removed: "place if have no power supervisor"
- moved on the sheet: C12, C13, C19, C20, C3, C4, C5, IC1, IC3, J1, JP4, JP6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
