File: pcb/skydrop.sch (EAGLE design)
At the start: 112 parts, among them IC1 RT9193-33GB, IC2 MCP73831/OT, IC3 STM809SWX6F, IC4 MS5611-01BA03, IC5 MCP23S17SO, Q1 BSS84, Q10 BSS84, Q2 BSS123, Q3 BSS123, Q4 BSS123, Q5 BSS84, Q6 BSS84, Q7 BSS123, Q8 BSS84, Q9 BSS84, SW1 431256083736, U2 W25Q16BVSS

Commit message: pcb
Connections:
- net N$25: now also OSC2.1; no longer OSC2.2
- net N$36: now also OSC2.2; no longer OSC2.1
Other:
- moved on the sheet: OSC2
Changed lines of the file:
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@@
 <attribute name="VALUE" x="-31.623" y="-128.27" size="1.778" layer="96" rot="R90"/>
 </instance>
-<instance part="OSC2" gate="G$1" x="147.32" y="-177.8" rot="R90"/>
+<instance part="OSC2" gate="G$1" x="147.32" y="-177.8" rot="R270"/>
 <instance part="JP1" gate="G$1" x="-157.48" y="-17.78" rot="MR270"/>
 <instance part="GND1" gate="1" x="-180.34" y="-45.72"/>
@@
 </segment>
 </net>
-<net name="N$25" class="0">
-<segment>
-<pinref part="UC1" gate="G$1" pin="PC14/OSC32_IN"/>
-<pinref part="OSC2" gate="G$1" pin="2"/>
-<wire x1="104.14" y1="-175.26" x2="147.32" y2="-175.26" width="0.1524" layer="91"/>
-<pinref part="C19" gate="G$1" pin="2"/>
-<wire x1="147.32" y1="-175.26" x2="152.4" y2="-175.26" width="0.1524" layer="91"/>
-<junction x="147.32" y="-175.26"/>
-</segment>
-</net>
 <net name="N$36" class="0">
 <segment>
-<pinref part="C20" gate="G$1" pin="2"/>
-<pinref part="OSC2" gate="G$1" pin="1"/>
-<wire x1="152.4" y1="-180.34" x2="147.32" y2="-180.34" width="0.1524" layer="91"/>
-<wire x1="147.32" y1="-180.34" x2="142.24" y2="-180.34" width="0.1524" layer="91"/>
 <wire x1="142.24" y1="-180.34" x2="142.24" y2="-177.8" width="0.1524" layer="91"/>
 <pinref part="UC1" gate="G$1" pin="PC15/OSC_OUT"/>
 <wire x1="142.24" y1="-177.8" x2="104.14" y2="-177.8" width="0.1524" layer="91"/>
+<pinref part="OSC2" gate="G$1" pin="2"/>
+<wire x1="142.24" y1="-180.34" x2="147.32" y2="-180.34" width="0.1524" layer="91"/>
+<pinref part="C20" gate="G$1" pin="2"/>
+<wire x1="147.32" y1="-180.34" x2="152.4" y2="-180.34" width="0.1524" layer="91"/>
 <junction x="147.32" y="-180.34"/>
 </segment>
@@
 </segment>
 </net>
+<net name="N$25" class="0">
+<segment>
+<pinref part="C19" gate="G$1" pin="2"/>
+<pinref part="OSC2" gate="G$1" pin="1"/>
+<wire x1="152.4" y1="-175.26" x2="147.32" y2="-175.26" width="0.1524" layer="91"/>
+<pinref part="UC1" gate="G$1" pin="PC14/OSC32_IN"/>
+<wire x1="147.32" y1="-175.26" x2="104.14" y2="-175.26" width="0.1524" layer="91"/>
+<junction x="147.32" y="-175.26"/>
+</segment>
+</net>
