File: pcb/skydrop.brd (EAGLE design)
At the start: 111.5 x 83 mm, 106 parts, among them IC1 RT9193-33GB, IC2 MCP73831/OT, IC3 STM809SWX6F, IC4 MS5611-01BA03, IC5 MCP23S17SO, Q1 BSS84, Q10 BSS84, Q2 BSS123, Q3 BSS123, Q4 BSS123, Q5 BSS84, Q6 BSS84, Q7 BSS123, Q8 BSS84, Q9 BSS84, U2 W25Q16BVSS

Commit message: [pcb] improve
Parts:
- removed BUT: BUT, SparkFun_20110922_my:TACTILE-SWITCH-1101NE
- added SW1: 431256083736, skydrop:431256083736
- added U$2: MPU-9250, invensense:LEAD-QFN24
- moved C12 6.02 mm to (53.2, 22.2)
- moved OSC 5.22 mm to (50.8, 24.2), turned to 180 degrees
- moved C13 4.03 mm to (53.2, 26.2)
- moved OSC2 3.61 mm to (47.0, 19.2), turned to 180 degrees
- moved JP4 2.69 mm to (40.0, 13.0)
- moved C8 2.61 mm to (49.8, 31.5), turned to 90 degrees
- moved R40 1.41 mm to (50.0, 47.2)
- moved C19 1.35 mm to (45.0, 25.2)
- moved C20 1.35 mm to (45.0, 23.2)
- moved C16 1.25 mm to (49.0, 44.5)
- moved D4 1.25 mm to (49.2, 39.2)
- moved R41 1.12 mm to (50.5, 41.8)
- moved C21 1.00 mm to (39.8, 45.8)
- moved R34 0.75 mm to (46.0, 39.2)
- moved C14 0.56 mm to (42.2, 27.2)
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Connections:
- removed net OSC32_IN_3: C19.2, OSC2.1, UC1.P$3
- removed net OSC32_OUT_4: C20.2, OSC2.4, UC1.P$4
- new net N$25: C19.2, OSC2.4, UC1.P$3
- new net N$36: C20.2, OSC2.1, UC1.P$4
- net GND: now also SW1.2; no longer BUT.P$2
- net N$11: now also SW1.3; no longer BUT.P$1
Routing:
- net BTN_C_T: track 67.7 -> 97.1 mm
- net OSC32_OUT_4: track 22.9 -> 0.00 mm
- net N$25: track 0.00 -> 21.9 mm
- net N$36: track 0.00 -> 19.2 mm
- net OSC32_IN_3: track 16.5 -> 0.00 mm
- net BTN_L_T: track 92.8 -> 100.7 mm
- net GND: track 405.7 -> 400.6 mm
- net N$11: track 6.79 -> 11.9 mm
- net OSC_OUT_6: track 13.9 -> 18.5 mm
- net VCC: track 185.2 -> 180.7 mm
- net OSC_IN_5: track 14.7 -> 18.1 mm
- net WAKE_UP: track 33.0 -> 36.2 mm
- net BTN_C_B: track 28.3 -> 25.4 mm
- net VCC_T: track 206.9 -> 209.1 mm
- net BTN_R_T: track 63.3 -> 65.5 mm
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Other:
- outline, holes or cut-outs redrawn

Commit message: [pcb] improve
Parts:
- added C29, C30: 0.1uF, skydrop:C0805
- added C7: 10nF, skydrop:C0805
- added R44, R45: 4.7k, skydrop:R0805
- R17, R18: value 4.7k -> 0; device skydrop:R0805 -> skydrop:R1206
- moved U$2 20.8 mm to (37.2, 18.6)
- moved IC4 20.3 mm to (54.0, 7.00)
- moved JP4 8.07 mm to (42.2, 5.25)
- moved Q10 6.52 mm to (28.0, 13.8)
- moved R37 6.52 mm to (28.0, 16.8)
- moved R38 6.39 mm to (28.5, 19.8), turned to 90 degrees
- moved R18 6.08 mm to (32.5, 22.6), turned to 90 degrees
- moved C18 5.76 mm to (35.6, 13.6), turned to 270 degrees
- moved R15 5.50 mm to (29.0, 9.25)
- moved R24 5.50 mm to (27.2, 9.25)
- moved R30 5.25 mm to (25.5, 9.25)
- moved JP6 5.10 mm to (15.5, 54.8)
- moved C17 4.60 mm to (14.0, 47.8)
- moved R28 4.60 mm to (21.2, 46.0)
- moved R31 4.60 mm to (14.0, 44.0)
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Connections:
- removed net MS5611_VCC: C18.1, IC4.P$1, IC4.P$2, IC4.P$4, IC4.P$5, R17.2, R18.2, UC1.P$57
- new net N$66: C29.1, U$2.10
- new net SENS_PWR: C18.1, C30.1, C7.1, IC4.P$1, IC4.P$2, IC4.P$4, IC4.P$5, R44.2, R45.2, U$2.1, U$2.13, U$2.22, U$2.8, UC1.P$57
- new net SENS_SCL: R18.1, R45.1, U$2.23, UC1.P$58
- new net SENS_SDA: R17.1, R44.1, U$2.24, UC1.P$59
- net GND: now also C29.2, C30.2, C7.2, U$2.11, U$2.18, U$2.20, U$2.9
- net MS5611_SCL: now also R18.2, U$2.7; no longer R17.1, UC1.P$58
- net MS5611_SDA: now also R17.2, U$2.21; no longer R18.1, UC1.P$59
Routing:
- net SENS_PWR: track 0.00 -> 54.7 mm, vias 0 -> 2
- net GND: track 400.6 -> 441.5 mm, vias 0 -> 2
- net N$22: track 20.6 -> 43.3 mm
- net MS5611_VCC: track 20.9 -> 0.00 mm
- net N$21: track 31.9 -> 48.1 mm
- net CHARGE_STAT: track 40.7 -> 49.1 mm
- net VCC: track 180.7 -> 188.7 mm
- net BAT_SNS: track 33.8 -> 41.7 mm
- net N$39: track 9.73 -> 4.13 mm
- net USB_CON: track 7.55 -> 12.9 mm
- net MS5611_SDA: track 8.85 -> 3.57 mm
- net MS5611_SCL: track 7.95 -> 2.70 mm
- net GPS_3D_FIX: track 35.3 -> 39.9 mm
- net GPS_PWR: track 56.5 -> 60.8 mm
- net FLASH_DO: track 18.4 -> 22.2 mm
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
Commit message: pcb
Parts:
- moved R1 4.07 mm to (17.2, 14.8)
- moved IC2 3.00 mm to (18.5, 10.0)
- moved C11 2.85 mm to (6.75, 19.2)
- moved C15 2.85 mm to (6.75, 21.2)
- moved C2 2.85 mm to (18.0, 19.2)
- moved C22 2.85 mm to (21.0, 21.8)
- moved C3 2.85 mm to (14.0, 30.8)
- moved C4 2.85 mm to (12.0, 30.8)
- moved C5 2.85 mm to (8.50, 30.8)
- moved D1 2.85 mm to (11.8, 18.0)
- moved D3 2.85 mm to (23.0, 28.8)
- moved IC1 2.85 mm to (7.00, 27.8)
- moved IC3 2.85 mm to (6.50, 24.0)
- moved Q1 2.85 mm to (11.2, 24.8)
- moved Q2 2.85 mm to (19.5, 26.2)
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Routing:
- net +5V: track 36.9 -> 41.9 mm
- net GND: track 441.5 -> 446.2 mm
- net N$21: track 48.1 -> 43.8 mm
- net N$27: track 6.34 -> 9.24 mm
- net SND_PWR: track 56.0 -> 53.9 mm
- net N$29: track 5.59 -> 7.62 mm
- net N$3: track 1.76 -> 3.75 mm
- net N$34: track 25.3 -> 23.3 mm
- net N$33: track 28.2 -> 26.2 mm
- net +UB: track 34.9 -> 33.4 mm
- net N$6: track 3.81 -> 5.19 mm
- net N$19: track 10.1 -> 11.4 mm
- net USB_VBUS: track 28.4 -> 29.7 mm
- net CHARGE_STAT: track 49.1 -> 47.8 mm
- net VCC: track 188.7 -> 187.8 mm
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
Commit message: pcb
Parts:
- moved OSC 12.3 mm to (45.8, 35.5), turned to 270 degrees
- moved R12 11.4 mm to (21.2, 68.8), turned to 180 degrees
- moved C13 11.3 mm to (46.8, 35.5)
- moved C12 10.7 mm to (46.8, 30.8)
- moved R11 9.41 mm to (17.2, 68.8), turned to 180 degrees
- moved D4 9.29 mm to (45.5, 47.8)
- moved C20 9.06 mm to (50.8, 30.2), turned to 180 degrees
- moved R2 8.84 mm to (12.8, 66.8)
- moved Q5 8.31 mm to (21.2, 65.8), turned to 180 degrees
- moved OSC2 8.05 mm to (50.5, 26.5), turned to 0 degrees
- moved R34 6.52 mm to (45.5, 45.8), turned to 180 degrees
- moved C19 6.27 mm to (50.8, 22.8), turned to 180 degrees
- moved Q3 5.50 mm to (7.00, 60.2)
- moved Q7 5.50 mm to (7.00, 56.5)
- moved R13 5.50 mm to (10.2, 56.5)
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Connections:
- net N$25: now also OSC2.1; no longer OSC2.4
- net N$36: now also OSC2.4; no longer OSC2.1
Routing:
- net GND: track 446.2 -> 422.9 mm
- net SND_PWR: track 53.9 -> 63.9 mm
- net OSC_IN_5: track 18.1 -> 9.30 mm
- net OSC_OUT_6: track 18.5 -> 10.1 mm
- net N$41: track 52.9 -> 46.1 mm
- net GPS_RX: track 31.5 -> 25.4 mm
- net GPS_3D_FIX: track 40.2 -> 34.3 mm
- net VCC: track 187.8 -> 193.7 mm
- net GPS_PWR: track 60.8 -> 55.3 mm
- net N$42: track 57.1 -> 52.1 mm
- net BAT_EN: track 26.0 -> 21.6 mm
- net WAKE_UP: track 35.6 -> 40.0 mm
- net N$25: track 21.9 -> 17.6 mm
- net BAT_SNS: track 41.2 -> 37.2 mm
- net LCD_DIN_B: track 23.3 -> 19.3 mm
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
Commit message: pcb
Parts:
- moved IC4 12.9 mm to (46.5, 17.5)
- moved C7 8.50 mm to (49.8, 10.2)
- moved D3 4.03 mm to (17.8, 28.0), turned to 180 degrees
- moved U$2 3.76 mm to (37.0, 14.8)
- moved C18 3.76 mm to (35.4, 9.85)
- moved C29 3.76 mm to (38.0, 9.85)
- moved C30 3.76 mm to (40.0, 9.85)
- moved R45 3.13 mm to (33.5, 28.5)
- moved R44 2.66 mm to (34.2, 26.8)
- moved C10 2.36 mm to (25.2, 45.5)
- moved R18 2.11 mm to (32.8, 24.8), turned to 180 degrees
- moved R16 2.02 mm to (25.0, 49.0)
- moved Q2 2.00 mm to (17.8, 31.5)
- moved R5 2.00 mm to (17.8, 34.5)
- moved R7 2.00 mm to (15.0, 33.5)
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Routing:
- net SENS_SCL: track 2.90 -> 19.7 mm
- net SENS_SDA: track 3.25 -> 16.2 mm
- net WAKE_UP: track 40.0 -> 44.4 mm
- net CHARGE_STAT: track 46.6 -> 49.8 mm
- net N$46: track 7.45 -> 5.10 mm
- net N$12: track 9.18 -> 11.3 mm
- net BAT_EN: track 21.6 -> 19.6 mm
- net N$37: track 28.8 -> 27.5 mm
- net N$35: track 7.77 -> 8.92 mm
- net +UB: track 36.1 -> 34.9 mm
- net N$32: track 1.96 -> 2.74 mm
- net VCC: track 193.7 -> 194.5 mm
- net GND: track 422.9 -> 423.7 mm
- net N$14: track 8.07 -> 7.41 mm
- net N$31: track 4.39 -> 4.93 mm
